File: keyboard.kicad_sch (KiCad schematic)
At the start: 0 parts

Commit message: full rework. ic numbers now same as in original schema
Parts:
- added C9: 0.1, Capacitor_THT:C_Radial_D5.0mm_H5.0mm_P2.00mm, symbol Device:C
- added R37, R38: 1k, Resistor_THT:R_Axial_DIN0204_L3.6mm_D1.6mm_P5.08mm_Horizontal, symbol Device:R
- added SW10: "7", symbol Switch:SW_Push
- added SW11: "8", symbol Switch:SW_Push
- added SW12: "9", symbol Switch:SW_Push
- added SW13: "A", symbol Switch:SW_Push
- added SW14: "B", symbol Switch:SW_Push
- added SW15: "C", symbol Switch:SW_Push
- added SW16: "D", symbol Switch:SW_Push
- added SW17: "E", symbol Switch:SW_Push
- added SW18: "F", symbol Switch:SW_Push
- added SW3: "0", symbol Switch:SW_Push
- added SW4: "1", symbol Switch:SW_Push
- added SW5: "2", symbol Switch:SW_Push
- added SW6: "3", symbol Switch:SW_Push
- added SW7: "4", symbol Switch:SW_Push
- added SW8: "5", symbol Switch:SW_Push
- added SW9: "6", symbol Switch:SW_Push
- added U11: 7401, symbol 74xx:74LS01
- added U15: 74LS01, symbol 74xx:74LS01
- added U19: 74LS27, symbol 74xx:74LS27
- added U21: 74LS04, Package_DIP:DIP-14_W7.62mm_LongPads, symbol 74xx:74LS04
- added U23: 74LS74, Package_DIP:DIP-14_W7.62mm_LongPads, symbol 74xx:74LS74
- added U24: 74LS32, Package_DIP:DIP-14_W7.62mm_LongPads, symbol 74xx:74LS32
- added U4: 7474, Package_DIP:DIP-14_W7.62mm, symbol 74xx:74LS74
- added U9: 7404, symbol 74xx:74LS04
Connections:
- new net: U23.11 (C), U23.3 (C), U24.3
- new net: R37.1, U23.13 (~{R}), U23.4 (~{S})
- new net: U23.5 (Q), U24.4
- new net: U24.13, U24.8
- new net: U24.9, U9.12
- new net: U24.11, U9.9
- new net: U23.9 (Q), U24.12
- new net +5V: R37.2, R38.2, U11.14 (VCC), U15.14 (VCC), U19.14 (VCC), U21.14 (VCC), U23.14 (VCC), U24.14 (VCC), U4.14 (VCC), U9.14 (VCC)
- new net A11: U9.13
- new net D2: U23.2 (D)
- new net D3: U23.12 (D)
- new net GND: C9.1, SW10.1, SW11.1, SW12.1, SW13.1, SW14.1, SW15.1, SW16.1, SW17.1, SW18.1, SW3.1, SW4.1, SW5.1, SW6.1, SW7.1, SW8.1, SW9.1, U11.7 (GND), U15.7 (GND), U19.7 (GND), U21.7 (GND), U23.7 (GND), U24.7 (GND), U4.7 (GND), U9.7 (GND)
- new net K0: SW3.2
- new net K1: SW4.2
- new net K2: SW5.2
- new net K3: SW6.2
- new net K4: SW7.2
- new net K5: SW8.2
- new net K6: SW9.2
- new net K7: SW10.2
- new net K8: SW11.2
- new net K9: SW12.2
- new net KA: SW13.2
- new net KB: SW14.2
- new net KC: SW15.2
- new net KD: SW16.2
- new net KE: SW17.2
- new net KF: SW18.2
- new net /0000h: U24.5
- new net /CSRAM: U9.8
- new net /CSROM: U24.6
- new net /E000h: U24.2
- new net /F000h: U24.10
- new net /JW: U24.1
- new net /R: C9.2, R38.1, U23.1 (~{R}), U23.10 (~{S})
- no-connect marks 0 -> 12
